Commit message: Last navigation version

File: noah_description/urdf/accurate_base_link.urdf.xacro (robot description, xacro)
@@ -316,4 +316,10 @@
 			<material>Gazebo/Blue</material>
 		</gazebo>
+		<joint name="imu_joint" type="fixed">
+			<parent link="front_link"/>
+			<child link="imu_link"/>
+			<origin xyz="0.0 0 0.068" rpy="0 0 0"/>
+		</joint>
+		<link name="imu_link"/>
 	</xacro:macro>
 </robot>

Commit message: Fix odometry publishing
Signed-off-by: Lucas Chiesa <lucas.chiesa@gmail.com>
Co-authored-by: Franco Cipollone <53065142+francocipollone@users.noreply.github.com>

File: noah_description/urdf/accurate_base_link.urdf.xacro (robot description, xacro)
@@ -8,4 +8,16 @@
 		<xacro:property name="M_PI" value="3.14159"/>
 		<!-- BASE************************************************************************** -->
+        <link name="base_footprint">
+            <!--
+            Dummy inertia-less link to prevent the following error:
+            [robot_state_publisher-1] The root link base_generic_link has an inertia specified in the URDF, but KDL does not support a root link with an inertia.
+            As a workaround, you can add an extra dummy link to your URDF.
+            -->
+        </link>
+        <joint name="base_frootprint_joint" type="fixed">
+            <parent link="base_footprint" />
+            <child link="base_generic_link" />
+            <origin xyz="0 0 0" rpy="0 0 0" />
+        </joint>
 		<xacro:property name="base_generic_depth" value="0.19"/>
 		<xacro:property name="base_generic_width" value="0.135"/>

File: noah_description/urdf/accurate_noah.urdf.xacro (robot description, xacro)
@@ -1,70 +1,62 @@
 <?xml version="1.0"?>
 <robot name="accurate_noah"
-	xmlns:xacro="http://www.ros.org/wiki/xacro">
-	<xacro:include filename="$(find noah_description)/urdf/materials.xacro" />
-	<xacro:include filename="$(find noah_description)/urdf/wheel.urdf.xacro" />
-	<xacro:include filename="$(find noah_description)/urdf/camera_sensor.urdf.xacro" />
-	<xacro:include filename="$(find noah_description)/urdf/accurate_base_link.urdf.xacro" />
-	<xacro:include filename="$(find noah_description)/urdf/caster_link.urdf.xacro" />
-	<xacro:property name="M_PI" value="3.14159"/>
-	<!-- Whole accurate_base_link dimensions -->
-	<xacro:property name="base_width" value="0.16426" />
-	<xacro:property name="base_depth" value="0.19" />
-	<xacro:property name="base_height" value="0.056" />
-	<xacro:property name="caster_radius" value="0.022" />
-	<xacro:property name="wheel_length" value="0.02" />
-	<xacro:property name="wheel_radius" value="0.05" />
-	<xacro:property name="camera_size" value="0.02" />
-	<!-- Base Link -->
-	<xacro:accurate_base_link />
-	<!-- Caster -->
-	<xacro:caster caster_radius="${caster_radius}" parent_link="caster_holder_link">
-		<origin xyz="0 0 0" rpy="0 0 0" />
-	</xacro:caster>
-	<!-- Wheels -->
-	<xacro:noah_wheel wheel_prefix="left" wheel_length="${wheel_length}" wheel_radius="${wheel_radius}" parent_link="left_wheel_adapter_link">
-		<origin xyz="0 ${wheel_length/2} 0" rpy="0 0 0" />
-	</xacro:noah_wheel>
-	<xacro:noah_wheel wheel_prefix="right" wheel_length="${wheel_length}" wheel_radius="${wheel_radius}" parent_link="right_wheel_adapter_link">
-		<origin xyz="0 -${wheel_length/2} 0" rpy="0 0 0" />
-	</xacro:noah_wheel>
-	<!-- Camera -->
-	<xacro:noah_camera camera_size="${camera_size}" parent_link="top_generic_link">
-		<!-- 0.0015 is half the heigth of top generic link -->
-		<origin xyz="${base_depth/3} 0 ${camera_size/2 + 0.0015}" rpy="0 0 0" />
-	</xacro:noah_camera>
-	<!-- *******Gazebo specific******* -->
-	<gazebo>
-    <!-- For ros2 we use gazebo_ros_joint_state_publisher instead of publishWheelJointState -->
-    <plugin name="joint_states" filename="libgazebo_ros_joint_state_publisher.so">
-      <joint_name>right_wheel_joint</joint_name>
-      <joint_name>left_wheel_joint</joint_name>
-    </plugin>
-		<plugin name="diff_drive" filename="libgazebo_ros_diff_drive.so">
-      <ros>
-        <namespace>/noah</namespace>
-        <!-- For the topics being published we would remap doing: -->
-        <!-- <argument>cmd_vel:=cmd_demo</argument> -->
-        <!-- <argument>odom:=odom_demo</argument> -->
-      </ros>
-      <!-- wheels -->
-      <left_joint>left_wheel_joint</left_joint>
-      <right_joint>right_wheel_joint</right_joint>
-      <!-- kinematics -->
-      <wheel_separation>1.25</wheel_separation>
-      <wheel_diameter>0.3</wheel_diameter>
-      <!-- limits -->
-      <max_wheel_torque>20</max_wheel_torque>
-      <max_wheel_acceleration>1.0</max_wheel_acceleration>
-      <!-- output -->
-			<update_rate>20</update_rate>
-      <publish_odom>true</publish_odom>
-      <publish_odom_tf>true</publish_odom_tf>
-      <odometry_frame>odom</odometry_frame>
-      <robot_base_frame>base_generic_link</robot_base_frame>
-			<command_topic>cmd_vel</command_topic>
-      <publish_wheel_tf>true</publish_wheel_tf>
-			<torque>20</torque>
-		</plugin>
-	</gazebo>
+    xmlns:xacro="http://www.ros.org/wiki/xacro">
+    <xacro:include filename="$(find noah_description)/urdf/materials.xacro" />
+    <xacro:include filename="$(find noah_description)/urdf/wheel.urdf.xacro" />
+    <xacro:include filename="$(find noah_description)/urdf/camera_sensor.urdf.xacro" />
+    <xacro:include filename="$(find noah_description)/urdf/accurate_base_link.urdf.xacro" />
+    <xacro:include filename="$(find noah_description)/urdf/caster_link.urdf.xacro" />
+    <xacro:property name="M_PI" value="3.14159" />
+    <!-- Whole accurate_base_link dimensions -->
+    <xacro:property name="base_width" value="0.16426" />
+    <xacro:property name="base_depth" value="0.19" />
+    <xacro:property name="base_height" value="0.056" />
+    <xacro:property name="caster_radius" value="0.022" />
+    <xacro:property name="wheel_length" value="0.02" />
+    <xacro:property name="wheel_radius" value="0.05" />
+    <xacro:property name="camera_size" value="0.02" />
+    <!-- Base Link -->
+    <xacro:accurate_base_link />
+    <!-- Caster -->
+    <xacro:caster caster_radius="${caster_radius}" parent_link="caster_holder_link">
+        <origin xyz="0 0 0" rpy="0 0 0" />
+    </xacro:caster>
+    <!-- Wheels -->
+    <xacro:noah_wheel wheel_prefix="left" wheel_length="${wheel_length}"
+        wheel_radius="${wheel_radius}" parent_link="left_wheel_adapter_link">
+        <origin xyz="0 ${wheel_length/2} 0" rpy="0 0 0" />
+    </xacro:noah_wheel>
+    <xacro:noah_wheel wheel_prefix="right" wheel_length="${wheel_length}"
+        wheel_radius="${wheel_radius}" parent_link="right_wheel_adapter_link">
+        <origin xyz="0 -${wheel_length/2} 0" rpy="0 0 0" />
+    </xacro:noah_wheel>
+    <!-- Camera -->
+    <xacro:noah_camera camera_size="${camera_size}" parent_link="top_generic_link">
+        <!-- 0.0015 is half the heigth of top generic link -->
+        <origin xyz="${base_depth/3} 0 ${camera_size/2 + 0.0015}" rpy="0 0 0" />
+    </xacro:noah_camera>
+    <!-- *******Gazebo specific******* -->
+    <gazebo>
+        <plugin name="diff_drive" filename="libgazebo_ros_diff_drive.so">
+            <ros>
+                <namespace>/noah</namespace>
+            </ros>
+            <!-- wheels -->
+            <left_joint>left_wheel_joint</left_joint>
+            <right_joint>right_wheel_joint</right_joint>
+            <!-- kinematics -->
+            <wheel_separation>1.25</wheel_separation>
+            <wheel_diameter>0.3</wheel_diameter>
+            <!-- limits -->
+            <max_wheel_torque>20</max_wheel_torque>
+            <max_wheel_acceleration>1.0</max_wheel_acceleration>
+            <!-- output -->
+            <update_rate>20</update_rate>
+            <publish_odom>true</publish_odom>
+            <publish_odom_tf>true</publish_odom_tf>
+            <odometry_frame>odom</odometry_frame>
+            <robot_base_frame>base_footprint</robot_base_frame>
+            <publish_wheel_tf>true</publish_wheel_tf>
+        </plugin>
+    </gazebo>
 </robot>

Commit message: Addressed Franco comments

File: noah_description/urdf/accurate_base_link.urdf.xacro (robot description, xacro)
@@ -316,10 +316,4 @@
 			<material>Gazebo/Blue</material>
 		</gazebo>
-		<joint name="imu_joint" type="fixed">
-			<parent link="front_link"/>
-			<child link="imu_link"/>
-			<origin xyz="0.0 0 0.068" rpy="0 0 0"/>
-		</joint>
-		<link name="imu_link"/>
 	</xacro:macro>
 </robot>

Commit message: Removed Gazebo tags from noah description
Signed-off-by: IDavGal <ignacio.davila@ekumenlabs.com>

File: noah_description/urdf/accurate_base_link.urdf.xacro (robot description, xacro)
@@ -41,7 +41,4 @@
 			</collision>
 		</link>
-		<gazebo reference="base_generic_link">
-			<material>Gazebo/SkyBlue</material>
-		</gazebo>
 		<!-- FRONT************************************************************************** -->
 		<xacro:property name="front_depth" value="0.06"/>
@@ -71,7 +68,4 @@
 			<origin xyz="${base_generic_depth/2 - front_depth/2} 0 ${front_heigth/2 + base_generic_heigth/2}" rpy="0 0 0" />
 		</joint>
-		<gazebo reference="front_link">
-			<material>Gazebo/SkyBlue</material>
-		</gazebo>
 		<!-- CASTER HOLDER************************************************************************** -->
 		<xacro:property name="caster_holder_radius" value="0.02299"/>
@@ -107,7 +101,4 @@
 			<!-- Origin in x adjusted by hand -->
 		</joint>
-		<gazebo reference="caster_holder_link">
-			<material>Gazebo/SkyBlue</material>
-		</gazebo>
 		<!-- BASE SUPPORTS************************************************************************** -->
 		<!-- Joints x and y coords are adjusted by hand -->
@@ -163,10 +154,4 @@
 			<origin xyz="-0.07847 0.04997 ${base_generic_heigth/2 + base_support_heigth/2}" rpy="0 0 0" />
 		</joint>
-		<gazebo reference="left_base_support_link">
-			<material>Gazebo/DarkGrey</material>
-		</gazebo>
-		<gazebo reference="right_base_support_link">
-			<material>Gazebo/DarkGrey</material>
-		</gazebo>
 		<!-- TOP************************************************************************** -->
 		<xacro:property name="top_generic_depth" value="0.19"/>
@@ -196,7 +181,4 @@
 			<origin xyz="0 0 ${base_support_heigth + top_generic_heigth/2 + base_generic_heigth/2}" rpy="0 0 0" />
 		</joint>
-		<gazebo reference="top_generic_link">
-			<material>Gazebo/SkyBlue</material>
-		</gazebo>
 		<!-- WHEEL ADAPTERS************************************************************************** -->
 		<xacro:property name="wheel_adapter_radius" value="0.01085"/>
@@ -250,10 +232,4 @@
 			<origin xyz="-${wheel_adapter_radius} -${front_width/2 + wheel_adapter_length/2} 0" rpy="0 0 0" />
 		</joint>
-		<gazebo reference="left_wheel_adapter_link">
-			<material>Gazebo/DarkGrey</material>
-		</gazebo>
-		<gazebo reference="right_wheel_adapter_link">
-			<material>Gazebo/DarkGrey</material>
-		</gazebo>
 		<!-- BATTERIES************************************************************************** -->
 		<xacro:property name="battery_depth" value="0.05"/>
@@ -283,7 +259,4 @@
 			<origin xyz="-${top_generic_depth/3} 0 ${battery_heigth/2 + top_generic_heigth/2}" rpy="0 0 0" />
 		</joint>
-		<gazebo reference="battery_link">
-			<material>Gazebo/Green</material>
-		</gazebo>
 		<!-- ELECTRONICS************************************************************************** -->
 		<xacro:property name="electronics_depth" value="0.08"/>
@@ -313,7 +286,4 @@
 			<origin xyz="-${electronics_depth/3.5} 0 ${base_generic_heigth/2 + electronics_heigth/2}" rpy="0 0 0" />
 		</joint>
-		<gazebo reference="electronics_link">
-			<material>Gazebo/Blue</material>
-		</gazebo>
 	</xacro:macro>
 </robot>

File: noah_description/urdf/accurate_noah.urdf.xacro (robot description, xacro)
@@ -37,26 +37,4 @@
     </xacro:noah_camera>
     <!-- *******Gazebo specific******* -->
-    <gazebo>
-        <plugin name="diff_drive" filename="libgazebo_ros_diff_drive.so">
-            <ros>
-                <namespace>/noah</namespace>
-            </ros>
-            <!-- wheels -->
-            <left_joint>left_wheel_joint</left_joint>
-            <right_joint>right_wheel_joint</right_joint>
-            <!-- kinematics -->
-            <wheel_separation>1.25</wheel_separation>
-            <wheel_diameter>0.3</wheel_diameter>
-            <!-- limits -->
-            <max_wheel_torque>20</max_wheel_torque>
-            <max_wheel_acceleration>1.0</max_wheel_acceleration>
-            <!-- output -->
-            <update_rate>20</update_rate>
-            <publish_odom>true</publish_odom>
-            <publish_odom_tf>true</publish_odom_tf>
-            <odometry_frame>odom</odometry_frame>
-            <robot_base_frame>base_footprint</robot_base_frame>
-            <publish_wheel_tf>true</publish_wheel_tf>
-        </plugin>
-    </gazebo>
+    <xacro:include filename="$(find noah_description)/urdf/gazebo_description.urdf.xacro" />
 </robot>

File: noah_description/urdf/camera_sensor.urdf.xacro (robot description, xacro)
@@ -63,84 +63,4 @@
       <origin xyz="0.0 0 0" rpy="-1.5707963267948966 0 -1.5707963267948966"/>
     </joint>
-    <gazebo reference="kinect">
-      <sensor name="kinect_camera" type="depth">
-        <!-- Set always_on only sensor, not on plugin -->
-        <always_on>0</always_on>
-        <!-- Set update_rate only sensor, not on plugin -->
-        <update_rate>20</update_rate>
-        <camera>
-          <horizontal_fov>1.047198</horizontal_fov>
-          <image>
-            <width>640</width>
-            <height>480</height>
-            <format>R8G8B8</format>
-          </image>
-          <distortion>
-            <k1>0.00000001</k1>
-            <k2>0.00000001</k2>
-            <k3>0.00000001</k3>
-            <p1>0.00000001</p1>
-            <p2>0.00000001</p2>
-            <center>0.0 0.0</center>
-          </distortion>
-          <clip>
-            <near>0.05</near>
-            <far>3</far>
-          </clip>
-        </camera>
-        <plugin name="kinect_plugin" filename="libgazebo_ros_camera.so">
-          <ros>
-            <namespace>noah</namespace>
-          </ros>
-          <!-- Set TF frame name. If empty, defaults to link name (i.e. "link_name") -->
-          <frame_name>kinect_gazebo</frame_name>
-          <!-- Set camera name. If empty, defaults to sensor name (i.e. "sensor_name") -->
-          <camera_name>kinect</camera_name>
-          <hack_baseline>0</hack_baseline>
-          <focal_length>0</focal_length>
-          <!-- No need to repeat distortion parameters or to set autoDistortion -->
-          <min_depth>0.5</min_depth>
-          <max_depth>3.0</max_depth>
-        </plugin>
-      </sensor>
-    </gazebo>
-    <gazebo reference="lens_link">
-      <sensor type="ray" name="head_hokuyo_sensor">
-        <pose>0 0 0 0 0 0</pose>
-        <visualize>true</visualize>
-        <update_rate>40</update_rate>
-        <ray>
-          <scan>
-            <horizontal>
-              <samples>720</samples>
-              <resolution>1</resolution>
-              <min_angle>-1.4</min_angle>
-              <max_angle>1.4</max_angle>
-            </horizontal>
-          </scan>
-          <range>
-            <min>0.10</min>
-            <max>30.0</max>
-            <resolution>0.01</resolution>
-          </range>
-          <noise>
-            <type>gaussian</type>
-            <mean>0.0</mean>
-            <stddev>0.01</stddev>
-          </noise>
-        </ray>
-        <plugin name="laser" filename="libgazebo_ros_ray_sensor.so">
-          <ros>
-            <namespace>/noah</namespace>
-            <remapping>~/out:=laser_scan</remapping>
-          </ros>
-          <output_type>sensor_msgs/LaserScan</output_type>
-        </plugin>
-      </sensor>
-    </gazebo>
-    <!-- Gazebo color -->
-    <gazebo reference="camera_link">
-      <material> Gazebo/Orange </material>
-    </gazebo>
   </xacro:macro>
 </robot>

File: noah_description/urdf/caster_link.urdf.xacro (robot description, xacro)
@@ -28,9 +28,4 @@
 		</joint>
 		<!-- caster gazebo properties -->
-		<gazebo reference="caster_link">
-			<mu1 value="0.0"/>
-			<mu2 value="0.0"/>
-			<material>Gazebo/DarkGrey</material>
-		</gazebo>
 	</xacro:macro>
 </robot>

File: noah_description/urdf/wheel.urdf.xacro (robot description, xacro)
@@ -35,12 +35,4 @@
 		</joint>
 		<!-- Wheels gazebo properties -->
-		<gazebo reference="${wheel_prefix}_wheel_link">
-			<mu1 value="1.0"/>
-			<mu2 value="1.0"/>
-			<kp value="10000000.0" />
-			<kd value="1.0" />
-			<fdir1 value="1 0 0"/>
-			<material>Gazebo/Black</material>
-		</gazebo>
 	</xacro:macro>
 </robot>
