Commit message: Remove inertia for caster in webots
Signed-off-by: IDavGal <ignacio.davila@ekumenlabs.com>

File: noah_description/urdf/accurate_noah.urdf.xacro (robot description, xacro)
@@ -8,4 +8,5 @@
     <xacro:include filename="$(find noah_description)/urdf/caster_link.urdf.xacro" />
     <xacro:property name="M_PI" value="3.14159" />
+    <xacro:property name="simulator" value="webots"/>
     <!-- Whole accurate_base_link dimensions -->
     <xacro:property name="base_width" value="0.16426" />

File: noah_description/urdf/caster_link.urdf.xacro (robot description, xacro)
@@ -4,8 +4,10 @@
 		<!-- caster description, simple sphere with no friction (ping pong ball) -->
 		<link name="caster_link">
-			<inertial>
-				<mass value="0.003" />
-				<inertia ixx="0.000000968" ixy="0" ixz="0" iyy="0.000000968" iyz="0" izz="0.000000968" />
-			</inertial>
+			<xacro:unless value="${simulator == 'webots'}">
+				<inertial>
+					<mass value="0.003" />
+					<inertia ixx="0.000000968" ixy="0" ixz="0" iyy="0.000000968" iyz="0" izz="0.000000968" />
+				</inertial>
+			</xacro:unless>
 			<visual>
 				<origin xyz="0 0 0" rpy="0 0 0" />
